Commit message: Minor adaptations for position of the ray and sensor mount

File: urdf/utils/custom_sensors.xacro (robot description, xacro)
@@ -54,5 +54,5 @@
                 <mass value="0" />
                 <origin rpy="0 0 0" xyz="0 0 0" />
-                <xacro:box_inertia mass="${mass}" x="${sensor_length}" y="${sensor_width}" z="${sensor_height}" />
+                <xacro:box_inertia mass="0.001" x="${sensor_length}" y="${sensor_width}" z="${sensor_height}" />
             </inertial>
         </link>
@@ -60,5 +60,5 @@
             <parent link="sensor_${id}_mount_point" />
             <child link="sensor_${id}" />
-            <origin xyz="0 0 0" rpy="0 0 1.57" />
+            <origin xyz="-${sensor_width / 2} 0 0" rpy="0 0 1.57" />
             <axis rpy="0 0 0" xyz="0 0 0"/>
         </joint>

Commit message: Default displacement for sensor

File: urdf/utils/custom_sensors.xacro (robot description, xacro)
@@ -9,6 +9,6 @@
     <xacro:property name="sensor_height" value="0.004" />
     <xacro:property name="originrpy" value="0 0 0" />
-    <xacro:property name="originxyz" value="0 0 0" />
-    <xacro:macro name="csensor" params="plink id mass originrpy originxyz jointxyz jointrpy">
+    <xacro:property name="originxyz" value="0 0 -0.003" />
+    <xacro:macro name="csensor" params="plink id mass jointxyz jointrpy">
         <link name="sensor_${id}_mount_point">
             <visual>
