Commit message: Single simu camera model

File: urdf/camera.urdf.xacro (robot description, xacro)
@@ -3,5 +3,4 @@
     <xacro:include filename="$(find ros_basics_models)/urdf/utils/inertia.xacro" />
     <xacro:property name="border_thickness" value="0.028"/>
-    <xacro:property name="z_mount" value="0.7"/>
     <xacro:property name="height" value="0.07"/>
     <xacro:property name="width" value="0.015"/>
@@ -10,7 +9,7 @@
     <joint name="world_joint" type="fixed">
         <parent link="world"/>
-        <child link="logi_c615"/>
+        <child link="simu_camera"/>
     </joint>
-    <link name="logi_c615">
+    <link name="simu_camera">
         <visual>
             <origin xyz="0 0 0" rpy="0 1.57 0"/>
@@ -30,5 +29,5 @@
         </inertial>
     </link>
-    <gazebo reference="logi_c615">
+    <gazebo reference="simu_camera">
         <sensor type="camera" name="top_camera">
             <pose>0 0 0 0 1.57 1.57</pose>
@@ -42,6 +41,6 @@
                 </image>
                 <clip>
-                    <near>0.02</near>
-                    <far>300</far>
+                    <near>0.5</near>
+                    <far>3</far>
                 </clip>
                 <noise>
@@ -56,5 +55,5 @@
                 <cameraName>robot_view</cameraName>
                 <imageTopicName>image_raw</imageTopicName>
-                <cameraInfoTopicName>logi_c615</cameraInfoTopicName>
+                <cameraInfoTopicName>simu_camera</cameraInfoTopicName>
                 <frameName>camera_link</frameName>
                 <hackBaseline>0.07</hackBaseline>
